Commit message: init omni sdf && remove joint relatives in sdf

File: dingo_simulator/dingo_gazebo/urdf/dingo-d.urdf.xacro (robot description, xacro)
@@ -159,4 +159,5 @@
   </joint>
   <link name="front_laser">
+    <origin xyz="0 0 0.085" rpy="0 0 0" /> <!-- TODO, not quite sure! -->
     <inertial>
       <mass value="1.1"/>
